File: Kicad/ESPower.kicad_pcb (KiCad board)
At the start: 2 copper layers, 84.6 x 14.5 mm, 35 parts, among them J1 Input, Q1 DMP2035U-7, Q2 FS8205A, SW2 A, SW3 B, U1 TP4056, U2 DW01A, U3 SPX3819M5-L-3-3, U4 TPS3839DBZ

Commit message: Updated labels
Parts:
- renumbered J1 to GND, Power to Switch
Other:
- board text removed: "Switch"

Commit message: Moved GND vias
Routing:
- net GND: track 51.9 -> 47.8 mm, vias 4 -> 5
Changed lines of the file:
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@@
     (effects (font (size 1 1) (thickness 0.15)))
   )
-  (via (at 110.617 96.139) (size 1.4) (drill 0.6) (layers F.Cu B.Cu) (net 1))
+  (via (at 108.458 99.822) (size 0.8) (drill 0.4) (layers F.Cu B.Cu) (net 1))
   (via (at 98.044 98.298) (size 0.8) (drill 0.4) (layers F.Cu B.Cu) (net 1))
   (via (at 93.472 104.14) (size 0.8) (drill 0.4) (layers F.Cu B.Cu) (net 1))
@@
   (segment (start 81.8134 95.123) (end 79.6544 97.282) (width 0.3) (layer F.Cu) (net 1))
   (segment (start 82.36 95.123) (end 81.8134 95.123) (width 0.3) (layer F.Cu) (net 1))
-  (segment (start 110.617 96.139) (end 113.411 96.139) (width 1.05) (layer F.Cu) (net 1))
   (segment (start 113.2255 95.9535) (end 113.411 96.139) (width 0.3) (layer F.Cu) (net 1))
   (segment (start 113.2255 95.814) (end 113.2255 95.9535) (width 0.3) (layer F.Cu) (net 1))
@@
   (segment (start 115.507 96.139) (end 115.951 95.695) (width 0.3) (layer F.Cu) (net 1))
   (segment (start 113.411 96.139) (end 115.507 96.139) (width 0.3) (layer F.Cu) (net 1))
-  (segment (start 106.947 99.187) (end 109.22 99.187) (width 0.3) (layer F.Cu) (net 1))
-  (segment (start 110.617 97.79) (end 110.617 96.139) (width 0.3) (layer F.Cu) (net 1))
-  (segment (start 109.22 99.187) (end 110.617 97.79) (width 0.3) (layer F.Cu) (net 1))
   (segment (start 149.159 96.967) (end 148.336 97.79) (width 0.3) (layer F.Cu) (net 1))
   (segment (start 151.908 96.967) (end 149.159 96.967) (width 0.3) (layer F.Cu) (net 1))
@@
   (segment (start 152.286 103.886) (end 151.638 103.238) (width 0.3) (layer F.Cu) (net 1))
   (segment (start 155.575 103.886) (end 152.286 103.886) (width 0.3) (layer F.Cu) (net 1))
+  (via (at 110.617 96.139) (size 1.4) (drill 0.6) (layers F.Cu B.Cu) (net 1))
+  (segment (start 110.617 96.139) (end 113.411 96.139) (width 1.05) (layer F.Cu) (net 1))
+  (segment (start 107.823 99.187) (end 108.458 99.822) (width 0.3) (layer F.Cu) (net 1))
+  (segment (start 106.947 99.187) (end 107.823 99.187) (width 0.3) (layer F.Cu) (net 1))
   (segment (start 106.376 105.664) (end 101.788 101.076) (width 1.4) (layer F.Cu) (net 2))
   (segment (start 106.986 105.664) (end 106.376 105.664) (width 1.4) (layer F.Cu) (net 2))
@@
   (segment (start 99.888 105.476) (end 100.076 105.664) (width 1.4) (layer F.Cu) (net 11))
   (segment (start 99.888 101.076) (end 99.888 105.476) (width 1.4) (layer F.Cu) (net 11))
-  (via (at 88.646 103.759) (size 0.8) (drill 0.4) (layers F.Cu B.Cu) (net 25))
+  (via (at 84.709 102.235) (size 0.8) (drill 0.4) (layers F.Cu B.Cu) (net 25))
 )
