File: Kicad/ESPower.sch (KiCad schematic (older format))
At the start: 35 parts, among them J1 Input, J2 Power Switch, J3 Output, J4 Battery, J5 GPIO, Q1 DMP2035U-7, Q2 FS8205A, SW1 PowerPath enable, SW2 A, SW3 B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

Commit message: Version 1.0
Parts:
- D1, D2: value SS34C -> SS34; footprint Diode_SMD:D_SMC -> Diode_SMD:D_SMA; symbol MBRS320T3:MBRS320T3 -> Device:D_Schottky; LCSC C13763 -> C8678
Connections:
- net +5V: now also D1.1 (K); no longer D1.C
- net at Q1.1, R1.1, SW1.2 (B): now also D2.2 (A); no longer D2.A
- net at C1.1, J2.1 (Pin_1), Q1.2: now also D2.1 (K); no longer D2.C
- net at J1.2 (Pin_2): now also D1.2 (A); no longer D1.A
Changed lines of the file:
@@
 $EndComp
 $Comp
-L MBRS320T3:MBRS320T3 D2
+L Device:D_Schottky D2
 U 1 1 62F7FF96
 P 4750 2000
-F 0 "D2" V 4704 2080 50  0000 L CNN
-F 1 "SS34C" V 4600 2050 50  0000 L CNN
-F 2 "Diode_SMD:D_SMC" H 4750 2000 50  0001 L BNN
+F 0 "D2" V 4750 1800 50  0000 L CNN
+F 1 "SS34" V 4650 1750 50  0000 L CNN
+F 2 "Diode_SMD:D_SMA" H 4750 2000 50  0001 L BNN
 F 3 "" H 4750 2000 50  0001 L BNN
-F 4 "C13763" V 4750 2000 50  0001 C CNN "LCSC"
+F 4 "C8678" V 4750 2000 50  0001 C CNN "LCSC"
 	1    4750 2000
-	0    1    1    0
+	0    -1   -1   0
 $EndComp
 $Comp
@@
 Wire Wire Line
 	4350 1700 4750 1700
-Wire Wire Line
-	4750 1700 4750 1800
 Connection ~ 4350 1700
-Wire Wire Line
-	4750 2200 4750 2300
 Connection ~ 4750 2300
 Wire Wire Line
@@
 	10550 4600 10150 4600
 $Comp
-L MBRS320T3:MBRS320T3 D1
+L Device:D_Schottky D1
 U 1 1 6317138C
 P 1550 1950
-F 0 "D1" H 1550 2167 50  0000 C CNN
-F 1 "SS34C" H 1550 2076 50  0000 C CNN
-F 2 "Diode_SMD:D_SMC" H 1550 1950 50  0001 L BNN
+F 0 "D1" H 1550 1700 50  0000 C CNN
+F 1 "SS34" H 1550 1800 50  0000 C CNN
+F 2 "Diode_SMD:D_SMA" H 1550 1950 50  0001 L BNN
 F 3 "" H 1550 1950 50  0001 L BNN
-F 4 "C13763" H 1550 1950 50  0001 C CNN "LCSC"
+F 4 "C8678" H 1550 1950 50  0001 C CNN "LCSC"
 	1    1550 1950
-	1    0    0    -1
+	-1   0    0    1
 $EndComp
 $Comp
@@
 	1    0    0    -1
 $EndComp
-Wire Wire Line
-	1750 1950 1900 1950
 Wire Wire Line
 	1900 1950 1900 1800
@@
 	1    0    0    -1
 $EndComp
-Wire Wire Line
-	1250 1950 1350 1950
 $Comp
 L Connector_Generic:Conn_01x02 J1
@@
 Wire Wire Line
 	4250 4250 4250 4350
+Wire Wire Line
+	1700 1950 1900 1950
+Wire Wire Line
+	1250 1950 1400 1950
+Wire Wire Line
+	4750 1700 4750 1850
+Wire Wire Line
+	4750 2150 4750 2300
 $EndSCHEMATC
